File: eagle_big/power_injector_rev_a.brd (EAGLE design)
At the start: 72.1 x 41.8 mm, 23 parts, among them J2 A00-108-220-450, J3 A00-108-220-450, X1 22-23-2041, X10 22-23-2041, X11 22-23-2041, X12 22-23-2041, X13 22-23-2041, X14 22-23-2041, X15 22-23-2041, X16 22-23-2041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

Commit message: Added terminators and changed connection sequence
Parts:
- added R1, R2: 120, rcl:R0805
- added TERM-L, TERM-R: 22-23-2021, con-molex:22-23-2021
Connections:
- new net N$11: R2.2, TERM-L.2
- new net N$3: R1.2, TERM-R.2
- net CANH: now also R2.1, TERM-R.1
- net CANL: now also R1.1, TERM-L.1
Routing:
- net CANH: track 196.3 -> 294.5 mm, vias 2 -> 0
- net POWER: track 242.7 -> 284.1 mm
- net CANL: track 226.8 -> 259.4 mm
- net N$11: track 0.00 -> 23.5 mm
- net N$3: track 0.00 -> 5.91 mm
- net +12V: track 18.6 -> 19.6 mm
Other:
- board text removed: "1"
- board text removed: "2"
- board text removed: "3"
