File: eagle_big/power_injector_rev_c.brd (EAGLE design)
At the start: 72.1 x 41.8 mm, 27 parts, among them J2 A00-108-220-450, J3 A00-108-220-450, X1 22-23-2041, X10 22-23-2041, X11 22-23-2041, X12 22-23-2041, X13 22-23-2041, X14 22-23-2041, X15 22-23-2041, X16 22-23-2041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

Commit message: Edit + bom added + gerbers
Parts:
- added U$1: (no value), seed_Logo:OSHW_FILLX100_NOTEXT
Changed lines of the file:
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@@
 <board>
 <plain>
-<text x="0.8" y="1" size="1.27" layer="25" font="fixed">Power Injector rev C</text>
-<text x="46.8" y="1.2" size="1.27" layer="25" font="fixed">www.grodansparadis.com</text>
-<text x="50.1" y="13.2" size="1.27" layer="25" font="fixed" rot="R90">PWR</text>
+<text x="0.6" y="0.8" size="1.27" layer="25">Power Injector rev C</text>
+<text x="47.5" y="0.9" size="1.27" layer="25">www.grodansparadis.com</text>
+<text x="50.2" y="12.4" size="1.27" layer="25" rot="R90">PWR</text>
 <wire x1="0" y1="0" x2="-0.06" y2="41.79" width="0" layer="20"/>
 <wire x1="-0.06" y1="41.79" x2="71.94" y2="41.79" width="0" layer="20"/>
@@
 <attribute name="NAME" x="32.1684" y="8.8366" size="0.6096" layer="25" font="fixed" ratio="10" rot="R270"/>
 </element>
-<element name="J4" library="con-jack-special" package="SPC4077" value="" x="27.1" y="12.6" rot="R90">
+<element name="J4" library="con-jack-special" package="SPC4077" value="" x="27.1" y="12.6" smashed="yes" rot="R90">
 <attribute name="MF" value="" x="27.1" y="12.6" size="1.778" layer="27" font="fixed" rot="R90" display="off"/>
 <attribute name="MPN" value="" x="27.1" y="12.6" size="1.778" layer="27" font="fixed" rot="R90" display="off"/>
 <attribute name="OC_FARNELL" value="unknown" x="27.1" y="12.6" size="1.778" layer="27" font="fixed" rot="R90" display="off"/>
 <attribute name="OC_NEWARK" value="unknown" x="27.1" y="12.6" size="1.778" layer="27" font="fixed" rot="R90" display="off"/>
+<attribute name="NAME" x="31.76" y="1.62" size="0.8128" layer="25" rot="R180"/>
+<attribute name="VALUE" x="33.45" y="2.44" size="1.27" layer="27" rot="R90"/>
 </element>
 <element name="X1" library="con-molex" package="22-23-2041" value="22-23-2041" x="5.85" y="24.16" smashed="yes" rot="R90">
@@
 <attribute name="NAME" x="42.96" y="9.81" size="0.8128" layer="25" ratio="10"/>
 </element>
+<element name="U$1" library="seed_Logo" package="OSHW_FILLX100_NOTEXT" value="" x="39.4" y="11.6"/>
 </elements>
 <signals>

Commit message: Named D1
Parts:
- D1: value PMEG3015EH,115 -> S1D
Changed lines of the file:
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@@
 <attribute name="NAME" x="50.94" y="3.78" size="0.6096" layer="25" font="fixed" rot="R270"/>
 </element>
-<element name="D1" library="diode" package="SMB" value="PMEG3015EH,115" x="37.32" y="16.68" smashed="yes" rot="R180">
+<element name="D1" library="diode" package="SMB" value="S1D" x="37.32" y="16.68" smashed="yes" rot="R180">
 <attribute name="NAME" x="37.979" y="14.551" size="0.6096" layer="25" font="fixed" rot="R180"/>
 </element>
