File: eagle_big/power_injector_rev_c.sch (EAGLE design)
At the start: 27 parts, among them J2 A00-108-220-450, J3 A00-108-220-450, X1 22-23-2041, X10 22-23-2041, X11 22-23-2041, X12 22-23-2041, X13 22-23-2041, X14 22-23-2041, X15 22-23-2041, X16 22-23-2041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

Commit message: Named D1
Parts:
- D1: value PMEG3015EH,115 -> S1D
Changed lines of the file:
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@@
 <part name="J3" library="vscpcan" deviceset="A00-108-220-450" device=""/>
 <part name="P+7" library="SUPPLY1" deviceset="+12V" device=""/>
-<part name="D1" library="diode" deviceset="DIODE-" device="SMB" value="PMEG3015EH,115"/>
+<part name="D1" library="diode" deviceset="DIODE-" device="SMB" value="S1D"/>
 <part name="GND3" library="SUPPLY1" deviceset="GND" device=""/>
 <part name="GND10" library="SUPPLY1" deviceset="GND" device=""/>
